File: hardware/PUYA_Prototype/PUYA_Prototype.kicad_sch (KiCad schematic)
At the start: 11 parts, among them J1 SWD, J2 L_Terminal, J3 R_Terminal, SW1 SW_RST, U1 PY32F002AA15M6TU, U2 AP2112K-3.3TRG1

Commit message: add pull-up resistor to NRST "DNP"
Parts:
- added R2: 10K, Resistor_SMD:R_0805_2012Metric, symbol Device:R_Small
Connections:
- net +3.3V: now also R2.2
- net NRST: now also R2.1
Changed lines of the file:
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@@
   (junction (at 247.65 63.5) (diameter 0) (color 0 0 0 0)
   )
+  (junction (at 48.641 148.59) (diameter 0) (color 0 0 0 0)
+  )
   (junction (at 232.41 49.53) (diameter 0) (color 0 0 0 0)
   )
@@
     (stroke (width 0) (type default))
   )
-  (wire (pts (xy 45.72 148.59) (xy 52.07 148.59))
+  (wire (pts (xy 45.72 148.59) (xy 48.641 148.59))
     (stroke (width 0) (type default))
   )
@@
   )
   (wire (pts (xy 50.8 123.19) (xy 50.8 127))
+    (stroke (width 0) (type default))
+  )
+  (wire (pts (xy 48.641 148.59) (xy 52.07 148.59))
     (stroke (width 0) (type default))
   )
@@
     (stroke (width 0) (type default))
   )
+  (wire (pts (xy 48.641 145.415) (xy 48.641 148.59))
+    (stroke (width 0) (type default))
+  )
   (text "Power Supply" (at 224.79 21.59 0)
     (effects (font (size 5 5)) (justify left bottom))
@@
         (path "/91c4888c-83fe-4d7b-b1c7-0dcb45a826cb"
           (reference "#PWR011") (unit 1)
+        )
+      )
+    )
+  )
+  (symbol (lib_id "power:+3.3V") (at 48.641 140.335 0) (unit 1)
+    (in_bom yes) (on_board yes) (dnp no) (fields_autoplaced)
+    (property "Reference" "#PWR015" (at 48.641 144.145 0)
+      (effects (font (size 1.27 1.27)) hide)
+    )
+    (property "Value" "+3.3V" (at 48.641 136.525 0)
+      (effects (font (size 1.27 1.27)))
+    )
+    (property "Footprint" "" (at 48.641 140.335 0)
+      (effects (font (size 1.27 1.27)) hide)
+    )
+    (property "Datasheet" "" (at 48.641 140.335 0)
+      (effects (font (size 1.27 1.27)) hide)
+    )
+    (pin "1")
+    (instances
+      (project "PUYA_Prototype"
+        (path "/91c4888c-83fe-4d7b-b1c7-0dcb45a826cb"
+          (reference "#PWR015") (unit 1)
         )
       )
@@
         )
       )
+    )
+  )
+  (symbol (lib_id "Device:R_Small") (at 48.641 142.875 180) (unit 1)
+    (in_bom yes) (on_board yes) (dnp yes) (fields_autoplaced)
+    (property "Reference" "R2" (at 50.8 142.24 0)
+      (effects (font (size 1.27 1.27)) (justify right))
+    )
+    (property "Value" "10K" (at 50.8 144.78 0)
+      (effects (font (size 1.27 1.27)) (justify right))
+    )
+    (property "Footprint" "Resistor_SMD:R_0805_2012Metric" (at 48.641 142.875 0)
+      (effects (font (size 1.27 1.27)) hide)
+    )
+    (property "Datasheet" "~" (at 48.641 142.875 0)
+      (effects (font (size 1.27 1.27)) hide)
+    )
+    (property "LCSC#" "C99198" (at 48.641 142.875 0)
+      (effects (font (size 1.27 1.27)) hide)
+    )
+    (property "manf#" "" (at 48.641 142.875 0)
+      (effects (font (size 1.27 1.27)) hide)
+    )
+    (pin "1")
+    (pin "2")
+    (instances
+      (project "PUYA_Prototype"
+        (path "/91c4888c-83fe-4d7b-b1c7-0dcb45a826cb"
+          (reference "R2") (unit 1)
+        )
+      )

Commit message: add library.pretty
Parts:
- U1: footprint Libraries:ESSOP10-EP -> PY32F002:PY32F002AA15M
Changed lines of the file:
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@@
       (effects (font (size 1.27 1.27)))
     )
-    (property "Footprint" "Libraries:ESSOP10-EP" (at 146.05 43.18 0)
+    (property "Footprint" "PY32F002:PY32F002AA15M" (at 146.05 43.18 0)
       (effects (font (size 1.27 1.27)) hide)
     )

Commit message: fix library
Parts:
- U1: footprint PY32F002:PY32F002AA15M -> Librarie:PY32F002AA15M
Changed lines of the file:
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@@
       (effects (font (size 1.27 1.27)))
     )
-    (property "Footprint" "PY32F002:PY32F002AA15M" (at 146.05 43.18 0)
+    (property "Footprint" "Librarie:PY32F002AA15M" (at 146.05 43.18 0)
       (effects (font (size 1.27 1.27)) hide)
     )
