File: hardware/PUYA_Prototype_PY32F030F28P6TU/PUYA_Prototype_PY32F030F28P6TU.kicad_sch (KiCad schematic)
At the start: 14 parts, among them J1 SWD, J2 Conn_01x10, J3 Conn_01x10, SW1 RESET, SW2 BOOT, U1 XC6220B331MR-G, U2 PY32F030F28P6TU

Commit message: feat(hw): add pcb design
Parts:
- SW1, SW2: footprint Button_Switch_SMD:SW_SPST_TL3342 -> Footprints:TS1088R02026
Connections:
- net BOOT: now also C4.2, R3.2, SW1.2; no longer C5.2, R1.2, SW2.2
- net PB5: now also U2.12 (PB5)
- net PB6: now also U2.13 (PB6)
- net PB7: now also U2.14 (PB7)
- net RST: now also C5.2, R1.2, SW2.2; no longer C4.2, R3.2, SW1.2
